File: emojipad_v2.brd (EAGLE design)
At the start: 99.2 x 85.1 mm, 60 parts, among them J1 ISP, SW1 CHERRY-MX-LED, SW10 CHERRY-MX-LED, SW11 CHERRY-MX-LED, SW12 CHERRY-MX-LED, SW13 CHERRY-MX-LED, SW14 CHERRY-MX-LED, SW15 CHERRY-MX-LED, SW16 CHERRY-MX-LED, SW2 CHERRY-MX-LED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

Commit message: Update to EmojiPad Sketch Files, Modification to V2 of the PCB: Changed pull-up to a GPIO pin, and D- to D12, Initial 3D Model Check In
Parts:
- moved C1 0.64 mm to (75.6, 44.5)
Connections:
- removed net MISO: J1.1, U1.18
- new net D7: U1.13
- net 5V: no longer R1.P$2
- net A0: now also R1.P$2
- net ROW3: now also J1.1, U1.18; no longer U1.13
Routing:
- net A0: track 0.00 -> 19.7 mm, vias 0 -> 1
- net MISO: track 16.1 -> 0.00 mm
- net 5V: track 136.0 -> 120.2 mm
- net A: track 222.6 -> 230.9 mm
- net COL3: track 99.3 -> 91.3 mm
- net ROW3: track 81.0 -> 86.4 mm, vias 0 -> 1
- net C: track 187.3 -> 185.0 mm
- net B: track 180.8 -> 183.0 mm
- net D: track 163.7 -> 161.9 mm
- net COL1: track 127.7 -> 128.5 mm
- net COL2: track 108.7 -> 109.4 mm
- net ROW2: track 93.8 -> 94.1 mm, vias 1 -> 0
- net GND: vias 10 -> 13
Other:
- board text added: "0.1uF"
- board text added: "1.5K"
- board text added: "100"
- board text added: "1K"
- board text added: "22pF"
- board text added: "3.6V"
- board text added: "68"
- board text added: "EmojiPad Rev 2, designed by Duncan Lowder"
- board text added: "EmojiPad V2"
- board text removed: "EmojiPad Rev 1A, designed by Duncan Lowder"
- board text removed: "EmojiPad V1"
